File: layout/pods.kicad_pcb (KiCad board)
At the start: 2 copper layers, 38.1 x 82.6 mm, 17 parts, among them J1 BATTERY, SW2 A, SW3 POWER, U1 STM32F103RCT6, U2 nRF24L01+, U3 MT-02, U4 ADP1710AUJZ, U5 SWD, U6 TP4056, U7 SH1106

Commit message: New PCB design
Parts:
- removed JP1: Jumper, Pin_Headers:Pin_Header_Straight_1x02_Pitch2.54mm
- removed REF** (x2): 1pin, Connectors:1pin
- removed SW2: A, Buttons_Switches_THT:SW_PUSH-12mm
- removed U3: MT-02, mt02:MT-02
- added BZ1: Buzzer, Connector_PinHeader_2.54mm:PinHeader_1x02_P2.54mm_Vertical, F.Cu at (119.7, 64.7)
- added C3: 100n, Capacitor_SMD:C_0805_2012Metric_Pad1.15x1.40mm_HandSolder, B.Cu at (106.9, 79.2)
- added C4: 100n, Capacitor_SMD:C_0805_2012Metric_Pad1.15x1.40mm_HandSolder, B.Cu at (106.9, 76.5)
- added C5: 100n, Capacitor_SMD:C_0805_2012Metric_Pad1.15x1.40mm_HandSolder, B.Cu at (111.9, 80.0)
- added C6: 100n, Capacitor_SMD:C_0805_2012Metric_Pad1.15x1.40mm_HandSolder, B.Cu at (111.9, 77.0)
- added C7: 100n, Capacitor_SMD:C_0805_2012Metric_Pad1.15x1.40mm_HandSolder, B.Cu at (111.9, 74.2)
- added JP_ID1: Jumper, Connector_PinHeader_2.54mm:PinHeader_1x02_P2.54mm_Vertical, F.Cu at (119.7, 74.5)
- added SW_A1: A, Button_Switch_THT:SW_TH_Tactile_Omron_B3F-10xx, F.Cu at (111.7, 103.0)
- added SW_DOWN1: A, Button_Switch_THT:SW_TH_Tactile_Omron_B3F-10xx, F.Cu at (88.2, 113.0)
- added SW_LEFT1: A, Button_Switch_THT:SW_TH_Tactile_Omron_B3F-10xx, F.Cu at (78.2, 103.0)
- added SW_RIGHT1: A, Button_Switch_THT:SW_TH_Tactile_Omron_B3F-10xx, F.Cu at (98.2, 103.0)
- added SW_UP1: A, Button_Switch_THT:SW_TH_Tactile_Omron_B3F-10xx, F.Cu at (88.2, 93.0)
- C1, C2: footprint Capacitors_SMD:C_0402_NoSilk -> Capacitor_SMD:C_0805_2012Metric_Pad1.15x1.40mm_HandSolder
- J1: footprint Pin_Headers:Pin_Header_Straight_1x02_Pitch2.54mm -> Connector_PinHeader_2.54mm:PinHeader_1x02_P2.54mm_Vertical; moved to B.Cu
- R1, R2: footprint Resistors_SMD:R_0805_HandSoldering -> Resistor_SMD:R_0805_2012Metric_Pad1.15x1.40mm_HandSolder
- SW3: footprint Pin_Headers:Pin_Header_Straight_1x03_Pitch2.54mm -> Connector_PinHeader_2.54mm:PinHeader_1x03_P2.54mm_Vertical
- U2: footprint RF_Modules:nRF24L01_Breakout -> Connector_PinHeader_2.54mm:PinHeader_2x04_P2.54mm_Vertical; moved to B.Cu
- U4: value ADP1710AUJZ -> ADP; footprint TO_SOT_Packages_SMD:TSOT-23-5 -> Package_TO_SOT_SMD:SOT-23-5_HandSoldering
- U5: footprint Pin_Headers:Pin_Header_Straight_1x04_Pitch2.54mm -> Connector_PinHeader_2.54mm:PinHeader_1x04_P2.54mm_Vertical
- U6: footprint tp4056 -> tp4056:tp4056; moved to B.Cu
- moved U4 76.3 mm to (83.2, 48.5), turned to 0 degrees
- moved C1 74.9 mm to (89.2, 48.5), turned to 90 degrees
- moved C2 64.7 mm to (93.7, 48.5), turned to 90 degrees
- moved SW3 64.4 mm to (77.7, 48.5)
- moved U2 63.7 mm to (76.7, 73.2)
- moved U1 55.8 mm to (98.7, 69.5)
- moved U6 52.3 mm to (98.7, 111.5), turned to 0 degrees
- moved U7 50.4 mm to (98.7, 68.5)
- moved R2 48.4 mm to (113.4, 58.0)
- moved R1 38.8 mm to (114.4, 48.7), turned to 90 degrees
- moved U5 33.8 mm to (119.7, 47.7), turned to 0 degrees
- moved J1 32.1 mm to (97.7, 95.0), turned to 270 degrees
Connections:
- U1 pad 1: Net-(U1-Pad1) -> (no net)
- U1 pad 11: Net-(U1-Pad11) -> (no net)
- U1 pad 12: Net-(U1-Pad12) -> (no net)
- U1 pad 13: Net-(U1-Pad13) -> (no net)
- U1 pad 14: Net-(U1-Pad14) -> (no net)
- U1 pad 15: Net-(U1-Pad15) -> (no net)
- U1 pad 16: Net-(U1-Pad16) -> (no net)
- U1 pad 17: Net-(U1-Pad17) -> (no net)
- U1 pad 26: Net-(U1-Pad26) -> (no net)
- U1 pad 27: Net-(U1-Pad27) -> (no net)
- U1 pad 28: Net-(U1-Pad28) -> (no net)
- U1 pad 29: Net-(U1-Pad29) -> (no net)
- U1 pad 3: BUTTON_B -> (no net)
- U1 pad 30: Net-(U1-Pad30) -> (no net)
- U1 pad 38: Net-(U1-Pad38) -> (no net)
- U1 pad 39: Net-(U1-Pad39) -> (no net)
- U1 pad 40: Net-(U1-Pad40) -> (no net)
- U1 pad 41: Net-(U1-Pad41) -> (no net)
- U1 pad 42: Net-(U1-Pad42) -> (no net)
- U1 pad 43: Net-(U1-Pad43) -> (no net)
- U1 pad 44: Net-(U1-Pad44) -> (no net)
- U1 pad 45: Net-(U1-Pad45) -> (no net)
- U1 pad 5: Net-(U1-Pad5) -> (no net)
- U1 pad 50: Net-(U1-Pad50) -> (no net)
- U1 pad 51: Net-(U1-Pad51) -> (no net)
- U1 pad 52: Net-(U1-Pad52) -> (no net)
- U1 pad 53: Net-(U1-Pad53) -> (no net)
- U1 pad 54: Net-(U1-Pad54) -> (no net)
- U1 pad 55: Net-(U1-Pad55) -> (no net)
- U1 pad 56: Net-(U1-Pad56) -> (no net)
- U1 pad 57: Net-(U1-Pad57) -> (no net)
- U1 pad 58: Net-(U1-Pad58) -> SOUND
- U1 pad 59: Net-(U1-Pad59) -> (no net)
- U1 pad 6: Net-(U1-Pad6) -> (no net)
- U1 pad 60: Net-(U1-Pad60) -> (no net)
- U1 pad 61: Net-(U1-Pad61) -> (no net)
- U1 pad 7: Net-(U1-Pad7) -> (no net)
- U4 pad 4: Net-(U4-Pad4) -> (no net)
- U6 pad 3: Net-(U6-Pad3) -> (no net)
- U6 pad 4: Net-(U6-Pad4) -> (no net)
Routing:
- net +3V3: track 210.6 -> 40.8 mm, vias 2 -> 5
- net GND: track 100.2 -> 43.2 mm, vias 2 -> 1
- net BUTTON_B: track 55.7 -> 0.00 mm
- net +4V: track 41.4 -> 88.5 mm, vias 0 -> 2
- net BUTTON_RIGHT: track 62.2 -> 34.3 mm, vias 0 -> 2
- net SWDIO: track 6.34 -> 27.6 mm
- net SOUND: track 0.00 -> 16.5 mm
- net SWCLK: track 8.76 -> 23.1 mm
- net Net-(SW3-Pad2): track 27.0 -> 14.1 mm
- net DEVICE_ID: track 4.99 -> 15.4 mm
- net BUTTON_UP: track 31.2 -> 21.1 mm
- net BUTTON_DOWN: track 39.0 -> 46.8 mm
- net BUTTON_LEFT: track 39.1 -> 33.5 mm
- net OLED_RES: track 10.8 -> 16.3 mm
- net NRF_IRQ: track 20.8 -> 15.3 mm
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- added copper zone on F.Cu, net +3V3
Other:
- board size 38.1 x 82.6 mm -> 50 x 80 mm
- board text removed: "BTN"
- board text removed: "JOYSTICK"
- board text removed: "USB"

Commit message: Updated kicad design
Parts:
- removed SW3: POWER, Connector_PinHeader_2.54mm:PinHeader_1x03_P2.54mm_Vertical
- added BRESET1: A, Button_Switch_THT:SW_TH_Tactile_Omron_B3F-10xx, F.Cu at (117.7, 86.5)
- added C8: 100n, Capacitor_SMD:C_0805_2012Metric_Pad1.15x1.40mm_HandSolder, B.Cu at (116.9, 89.7)
- added R3: 10K, Resistor_SMD:R_0805_2012Metric_Pad1.15x1.40mm_HandSolder, B.Cu at (121.4, 89.7)
- added R4: 10K, Resistor_SMD:R_0805_2012Metric_Pad1.15x1.40mm_HandSolder, B.Cu at (119.7, 50.5)
- added R5: 10K, Resistor_SMD:R_0805_2012Metric_Pad1.15x1.40mm_HandSolder, B.Cu at (119.7, 47.0)
- added SW_POW1: POWER, Connector_Wire:SolderWirePad_1x03_P3.175mm_Drill0.8mm, F.Cu at (77.4, 48.0)
- BZ1, JP_ID1: footprint Connector_PinHeader_2.54mm:PinHeader_1x02_P2.54mm_Vertical -> Connector_Wire:SolderWirePad_1x02_P3.81mm_Drill0.8mm
- J1: footprint Connector_PinHeader_2.54mm:PinHeader_1x02_P2.54mm_Vertical -> Connector_Wire:SolderWirePad_1x02_P3.81mm_Drill0.8mm; moved to F.Cu
- U2: footprint Connector_PinHeader_2.54mm:PinHeader_2x04_P2.54mm_Vertical -> nrf24:NRF24L01; moved to F.Cu
- U4: value ADP -> ADP1710AUJZ
- U5: footprint Connector_PinHeader_2.54mm:PinHeader_1x04_P2.54mm_Vertical -> Connector_PinSocket_2.54mm:PinSocket_2x03_P2.54mm_Vertical
- U6: moved to F.Cu
- moved C6 24.3 mm to (87.9, 80.7)
- moved C7 24.3 mm to (87.9, 78.0)
- moved J1 23.0 mm to (88.9, 116.2)
- moved C5 20.3 mm to (106.4, 60.5), turned to 0 degrees
- moved U6 12.8 mm to (110.7, 116.0), turned to 270 degrees
- moved U5 10.0 mm to (109.7, 47.0), turned to 90 degrees
- moved R1 9.51 mm to (104.9, 48.2)
- moved U2 9.02 mm to (74.9, 64.4), turned to 90 degrees
- moved SW_A1 5.00 mm to (111.7, 98.0)
- moved SW_DOWN1 5.00 mm to (88.2, 108.0)
- moved SW_LEFT1 5.00 mm to (78.2, 98.0)
- moved SW_RIGHT1 5.00 mm to (98.2, 98.0)
- moved SW_UP1 5.00 mm to (88.2, 88.0)
- moved C3 4.85 mm to (110.9, 76.5), turned to 270 degrees
- moved BZ1 1.40 mm to (119.6, 63.3), turned to 270 degrees
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Connections:
- U1 pad 1: (no net) -> +3V3
- U1 pad 12: (no net) -> GND
- U1 pad 13: (no net) -> +3V3
- U1 pad 55: (no net) -> SWO
- U1 pad 7: (no net) -> RESET
Routing:
- net RESET: track 0.00 -> 75.3 mm, vias 0 -> 4
- net +3V3: track 40.8 -> 82.9 mm, vias 5 -> 8
- net SWO: track 0.00 -> 34.2 mm
- net GND: track 43.2 -> 66.7 mm, vias 1 -> 4
- net +4V: track 88.5 -> 109.5 mm, vias 2 -> 0
- net BUTTON_DOWN: track 46.8 -> 36.4 mm
- net NRF_SCK: track 19.2 -> 26.5 mm
- net BUTTON_RIGHT: track 34.3 -> 28.0 mm
- net -BATT: track 6.31 -> 12.1 mm
- net BUTTON_UP: track 21.1 -> 15.4 mm
- net BUTTON_A: track 34.9 -> 29.5 mm
- net +BATT: track 6.63 -> 10.3 mm
- net SWDIO: track 27.6 -> 23.9 mm
- net NRF_IRQ: track 15.3 -> 17.6 mm, vias 0 -> 2
- net SWCLK: track 23.1 -> 25.2 mm
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
Commit message: Updated schematic/pcb
Parts:
- removed R4: 10K, Resistor_SMD:R_0805_2012Metric_Pad1.15x1.40mm_HandSolder
- added REF**: MountingHole_3.2mm_M3, MountingHole:MountingHole_3.2mm_M3, F.Cu at (116.7, 54.5)
- added REF**: MountingHole_3.2mm_M3, MountingHole:MountingHole_3.2mm_M3, F.Cu at (74.7, 54.5)
- added REF**: MountingHole_3.2mm_M3, MountingHole:MountingHole_3.2mm_M3, F.Cu at (74.7, 136.5)
- added REF**: MountingHole_3.2mm_M3, MountingHole:MountingHole_3.2mm_M3, F.Cu at (116.7, 136.5)
- BRESET1, SW_A1, SW_DOWN1, SW_LEFT1, SW_RIGHT1, SW_UP1: footprint Button_Switch_THT:SW_TH_Tactile_Omron_B3F-10xx -> switches:SW_TH_Tactile_Omron_Fixed
- U5: footprint Connector_PinSocket_2.54mm:PinSocket_2x03_P2.54mm_Vertical -> Connector_PinHeader_2.54mm:PinHeader_2x03_P2.54mm_Horizontal
- moved SW_POW1 88.8 mm to (80.5, 136.7), turned to 0 degrees
- moved C2 85.4 mm to (85.4, 133.5), turned to 180 degrees
- moved C1 81.5 mm to (78.2, 129.2)
- moved U4 79.8 mm to (83.7, 128.2)
- moved R5 22.2 mm to (116.7, 69.0)
- moved R2 12.7 mm to (107.9, 69.5), turned to 0 degrees
- moved U5 12.0 mm to (110.2, 59.0), turned to 180 degrees
- moved C7 11.8 mm to (86.7, 89.7), turned to 270 degrees
- moved BZ1 11.4 mm to (116.6, 74.3)
- moved C3 11.4 mm to (107.9, 87.5), turned to 90 degrees
- moved C4 11.4 mm to (103.9, 87.5), turned to 90 degrees
- moved C8 11.4 mm to (113.9, 100.7)
- moved JP_ID1 11.4 mm to (116.6, 86.6)
- moved R1 11.4 mm to (101.9, 59.2)
- moved R3 11.4 mm to (118.4, 100.7)
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Connections:
- U1 pad 18: +3V3 -> GND
- U1 pad 19: GND -> +3V3
- U1 pad 31: +3V3 -> GND
- U1 pad 32: GND -> +3V3
- U1 pad 47: +3V3 -> GND
- U1 pad 48: GND -> +3V3
- U1 pad 63: +3V3 -> GND
- U1 pad 64: GND -> +3V3
Routing:
- net +4V: track 109.5 -> 29.3 mm, vias 0 -> 1
- net RESET: track 75.3 -> 89.8 mm
- net GND: track 66.7 -> 53.6 mm, vias 4 -> 5
- net +BATT: track 10.3 -> 20.7 mm
- net BUTTON_UP: track 15.4 -> 21.9 mm
- net BUTTON_RIGHT: track 28.0 -> 34.5 mm
- net BUTTON_LEFT: track 31.6 -> 38.1 mm
- net BUTTON_DOWN: track 36.4 -> 42.9 mm
- net BUTTON_A: track 29.5 -> 36.0 mm
- net SWCLK: track 25.2 -> 30.6 mm
- net +3V3: track 82.9 -> 88.2 mm
- net -BATT: track 12.1 -> 15.5 mm
- net SWO: track 34.2 -> 37.4 mm, vias 0 -> 1
- net SWDIO: track 23.9 -> 25.3 mm
- net Net-(SW_POW1-Pad2): track 14.1 -> 13.1 mm, vias 0 -> 2
Other:
- board size 50 x 80 mm -> 50 x 90 mm
- board text added: "PODS v2 2018 @desertkun"
