File: layout/pods.sch (KiCad schematic (older format))
At the start: 15 parts, among them J1 BATTERY, SW2 A, SW3 POWER, U1 STM32F103RCT6, U2 nRF24L01+, U3 MT-02, U4 ADP1710AUJZ, U5 SWD, U6 TP4056, U7 SH1106

Commit message: New PCB design
Parts:
- removed U3: MT-02, symbol MT-02
- added BZ1: Buzzer, Connector_PinHeader_2.54mm:PinHeader_1x02_P2.54mm_Vertical, symbol Device:Buzzer
- added C3, C4, C5, C6, C7: 100n, Capacitor_SMD:C_0805_2012Metric_Pad1.15x1.40mm_HandSolder, symbol pods-rescue:C
- added SW_DOWN1, SW_LEFT1, SW_RIGHT1, SW_UP1: A, Button_Switch_THT:SW_TH_Tactile_Omron_B3F-10xx, symbol pods-rescue:SW_Push
- C1, C2: footprint Capacitors_SMD:C_0402_NoSilk -> Capacitor_SMD:C_0805_2012Metric_Pad1.15x1.40mm_HandSolder; symbol C -> pods-rescue:C
- J1: footprint Pin_Headers:Pin_Header_Straight_1x02_Pitch2.54mm -> Connector_PinHeader_2.54mm:PinHeader_1x02_P2.54mm_Vertical; symbol Conn_01x02 -> pods-rescue:Conn_01x02
- JP_ID1: renamed from JP1; footprint Pin_Headers:Pin_Header_Straight_1x02_Pitch2.54mm -> Connector_PinHeader_2.54mm:PinHeader_1x02_P2.54mm_Vertical; symbol Jumper -> pods-rescue:Jumper
- R1, R2: footprint Resistors_SMD:R_0805_HandSoldering -> Resistor_SMD:R_0805_2012Metric_Pad1.15x1.40mm_HandSolder; symbol R -> pods-rescue:R
- SW3: footprint Pin_Headers:Pin_Header_Straight_1x03_Pitch2.54mm -> Connector_PinHeader_2.54mm:PinHeader_1x03_P2.54mm_Vertical; symbol SW_SPDT -> pods-rescue:SW_SPDT
- SW_A1: renamed from SW2; footprint Buttons_Switches_THT:SW_PUSH-12mm -> Button_Switch_THT:SW_TH_Tactile_Omron_B3F-10xx; symbol SW_Push -> pods-rescue:SW_Push
- U1: symbol STM32F103RCT6 -> pods-rescue:STM32F103RCT6
- U2: footprint RF_Modules:nRF24L01_Breakout -> Connector_PinHeader_2.54mm:PinHeader_2x04_P2.54mm_Vertical; symbol nRF24L01+ -> pods-rescue:nRF24L01+
- U4: footprint TO_SOT_Packages_SMD:TSOT-23-5 -> Package_TO_SOT_SMD:SOT-23-5_HandSoldering; symbol ADP1710AUJZ -> pods-rescue:ADP1710AUJZ
- U5: footprint (none) -> Connector_PinHeader_2.54mm:PinHeader_1x04_P2.54mm_Vertical; symbol SWD -> pods-rescue:SWD
- U6: symbol TP4056 -> pods-rescue:TP4056
- U7: symbol SH1106 -> pods-rescue:SH1106
Connections:
- net +3V3: now also C3.1, C4.1, C5.1, C6.1, C7.1
- net BUTTON_DOWN: now also SW_DOWN1.2
- net BUTTON_LEFT: now also SW_LEFT1.2
- net BUTTON_RIGHT: now also SW_RIGHT1.2
- net BUTTON_UP: now also SW_UP1.2
- net GND: now also BZ1.1 (-), C3.2, C4.2, C5.2, C6.2, C7.2, SW_DOWN1.1, SW_LEFT1.1, SW_RIGHT1.1, SW_UP1.1; no longer U5.6 (RST)
- net SOUND: now reaches U1.58 (PB6/I2C1_SCL/TIM4_CH1/USART1_TX)
- net SOUND: now also BZ1.2 (+)
- net BUTTON_B: no longer names the net of U1.3 (PC14/OSC32_IN)
- no-connect marks 5 -> 39
Other:
- moved on the sheet: JP_ID1, SW_A1, U5

Commit message: Updated kicad design
Parts:
- added BRESET1: A, Button_Switch_THT:SW_TH_Tactile_Omron_B3F-10xx, symbol pods-rescue:SW_Push
- added C8: 100n, Capacitor_SMD:C_0805_2012Metric_Pad1.15x1.40mm_HandSolder, symbol pods-rescue:C
- added R3, R4, R5: 10K, Resistor_SMD:R_0805_2012Metric_Pad1.15x1.40mm_HandSolder, symbol pods-rescue:R
- BZ1, J1, JP_ID1: footprint Connector_PinHeader_2.54mm:PinHeader_1x02_P2.54mm_Vertical -> Connector_Wire:SolderWirePad_1x02_P3.81mm_Drill0.8mm
- SW_POW1: renamed from SW3; footprint Connector_PinHeader_2.54mm:PinHeader_1x03_P2.54mm_Vertical -> Connector_Wire:SolderWirePad_1x03_P3.175mm_Drill0.8mm
- U2: footprint Connector_PinHeader_2.54mm:PinHeader_2x04_P2.54mm_Vertical -> nrf24:NRF24L01
- U5: footprint Connector_PinHeader_2.54mm:PinHeader_1x04_P2.54mm_Vertical -> Connector_PinSocket_2.54mm:PinSocket_2x03_P2.54mm_Vertical
Connections:
- net +3V3: now also U1.1 (VBAT), U1.13 (VDDA), R3.2, R4.1, R5.1
- net GND: now also U1.12 (VSSA), BRESET1.2, C8.1
- net SWO: now reaches U1.55 (JTDO/SPI3_SCK/I2S3_CK/TIM2_CH2/PB3/TRACESWO/SPI1_SCK)
- net SWO: now also U5.5 (SWO), R5.2
- net RESET: now reaches U1.7 (NRST)
- net RESET: now also U5.6 (RST), BRESET1.1, C8.2, R3.1, R4.2
- no-connect marks 39 -> 34
Other:
- moved on the sheet: R1, R2, U5, U7

Commit message: Updated schematic/pcb
Parts:
- removed R4: 10K, Resistor_SMD:R_0805_2012Metric_Pad1.15x1.40mm_HandSolder, symbol pods-rescue:R
- BRESET1, SW_A1, SW_DOWN1, SW_LEFT1, SW_RIGHT1, SW_UP1: footprint Button_Switch_THT:SW_TH_Tactile_Omron_B3F-10xx -> switches:SW_TH_Tactile_Omron_Fixed
- U5: footprint Connector_PinSocket_2.54mm:PinSocket_2x03_P2.54mm_Vertical -> Connector_PinHeader_2.54mm:PinHeader_2x03_P2.54mm_Horizontal
Connections:
- net +3V3: now also U1.19 (VDD_4), U1.32 (VDD_1), U1.48 (VDD_2), U1.64 (VDD_3); no longer U1.18 (VSS_4), U1.31 (VSS_1), U1.47 (VSS_2), U1.63 (VSS_3)
- net GND: now also U1.18 (VSS_4), U1.31 (VSS_1), U1.47 (VSS_2), U1.63 (VSS_3); no longer U1.19 (VDD_4), U1.32 (VDD_1), U1.48 (VDD_2), U1.64 (VDD_3)
Changed lines of the file:
@@
 L power:GND #PWR0108
 U 1 1 5C04BC99
-P 4050 3500
-F 0 "#PWR0108" H 4050 3250 50  0001 C CNN
-F 1 "GND" H 4055 3327 50  0000 C CNN
-F 2 "" H 4050 3500 50  0001 C CNN
-F 3 "" H 4050 3500 50  0001 C CNN
-	1    4050 3500
+P 3850 4000
+F 0 "#PWR0108" H 3850 3750 50  0001 C CNN
+F 1 "GND" H 3855 3827 50  0000 C CNN
+F 2 "" H 3850 4000 50  0001 C CNN
+F 3 "" H 3850 4000 50  0001 C CNN
+	1    3850 4000
 	1    0    0    -1
 $EndComp
 Wire Wire Line
 	4300 3400 4300 3500
-Wire Wire Line
-	4050 3400 4300 3400
-Wire Wire Line
-	4050 3500 4050 3400
 $Comp
 L power:+3.3V #PWR0104
 U 1 1 5C04B8EE
-P 4050 4000
-F 0 "#PWR0104" H 4050 3850 50  0001 C CNN
-F 1 "+3.3V" H 4065 4173 50  0000 C CNN
-F 2 "" H 4050 4000 50  0001 C CNN
-F 3 "" H 4050 4000 50  0001 C CNN
-	1    4050 4000
+P 3950 3400
+F 0 "#PWR0104" H 3950 3250 50  0001 C CNN
+F 1 "+3.3V" H 3965 3573 50  0000 C CNN
+F 2 "" H 3950 3400 50  0001 C CNN
+F 3 "" H 3950 3400 50  0001 C CNN
+	1    3950 3400
 	1    0    0    -1
 $EndComp
@@
 	4100 4000 4100 4100
 Connection ~ 4100 4000
-Wire Wire Line
-	4050 4000 4100 4000
 Text GLabel 9050 1900 2    60   Input ~ 0
 DEVICE_ID
@@
 F 0 "SW_DOWN1" H 1950 2450 50  0000 L CNN
 F 1 "A" H 1900 2290 50  0000 C CNN
-F 2 "Button_Switch_THT:SW_TH_Tactile_Omron_B3F-10xx" H 1900 2550 50  0001 C CNN
+F 2 "switches:SW_TH_Tactile_Omron_Fixed" H 1900 2550 50  0001 C CNN
 F 3 "" H 1900 2550 50  0001 C CNN
 	1    1900 2350
@@
 F 0 "SW_UP1" H 1950 2150 50  0000 L CNN
 F 1 "A" H 1900 1990 50  0000 C CNN
-F 2 "Button_Switch_THT:SW_TH_Tactile_Omron_B3F-10xx" H 1900 2250 50  0001 C CNN
+F 2 "switches:SW_TH_Tactile_Omron_Fixed" H 1900 2250 50  0001 C CNN
 F 3 "" H 1900 2250 50  0001 C CNN
 	1    1900 2050
@@
 F 0 "SW_RIGHT1" H 1950 1850 50  0000 L CNN
 F 1 "A" H 1900 1690 50  0000 C CNN
-F 2 "Button_Switch_THT:SW_TH_Tactile_Omron_B3F-10xx" H 1900 1950 50  0001 C CNN
+F 2 "switches:SW_TH_Tactile_Omron_Fixed" H 1900 1950 50  0001 C CNN
 F 3 "" H 1900 1950 50  0001 C CNN
 	1    1900 1750
@@
 F 0 "SW_LEFT1" H 1950 1550 50  0000 L CNN
 F 1 "A" H 1900 1390 50  0000 C CNN
-F 2 "Button_Switch_THT:SW_TH_Tactile_Omron_B3F-10xx" H 1900 1650 50  0001 C CNN
+F 2 "switches:SW_TH_Tactile_Omron_Fixed" H 1900 1650 50  0001 C CNN
 F 3 "" H 1900 1650 50  0001 C CNN
 	1    1900 1450
@@
 F 0 "SW_A1" H 1950 1200 50  0000 L CNN
 F 1 "A" H 1900 1040 50  0000 C CNN
-F 2 "Button_Switch_THT:SW_TH_Tactile_Omron_B3F-10xx" H 1900 1300 50  0001 C CNN
+F 2 "switches:SW_TH_Tactile_Omron_Fixed" H 1900 1300 50  0001 C CNN
 F 3 "" H 1900 1300 50  0001 C CNN
 	1    1900 1100
@@
 F 0 "U5" H 6950 5300 60  0000 C CNN
 F 1 "SWD" H 7050 4500 60  0000 C CNN
-F 2 "Connector_PinSocket_2.54mm:PinSocket_2x03_P2.54mm_Vertical" H 7050 5000 60  0001 C CNN
+F 2 "Connector_PinHeader_2.54mm:PinHeader_2x03_P2.54mm_Horizontal" H 7050 5000 60  0001 C CNN
 F 3 "" H 7050 5000 60  0001 C CNN
 	1    7050 5000
@@
 NoConn ~ 9050 3900
 NoConn ~ 9050 4100
-Wire Wire Line
-	4850 3900 4300 3900
-Wire Wire Line
-	4300 3900 4300 3800
-Connection ~ 4300 3800
-$Comp
-L power:+3.3V #PWR01
-U 1 1 5C0199E3
-P 4350 3250
-F 0 "#PWR01" H 4350 3100 50  0001 C CNN
-F 1 "+3.3V" H 4365 3423 50  0000 C CNN
-F 2 "" H 4350 3250 50  0001 C CNN
-F 3 "" H 4350 3250 50  0001 C CNN
-	1    4350 3250
-	1    0    0    -1
-$EndComp
-Wire Wire Line
-	4850 3300 4350 3300
-Wire Wire Line
-	4350 3300 4350 3250
-Wire Wire Line
-	4850 3400 4350 3400
-Wire Wire Line
-	4350 3400 4350 3300
-Connection ~ 4350 3300
 $Comp
 L power:GND #PWR04
@@
 F 0 "BRESET1" H 8300 6950 50  0000 L CNN
 F 1 "A" H 8250 6790 50  0000 C CNN
-F 2 "Button_Switch_THT:SW_TH_Tactile_Omron_B3F-10xx" H 8250 7050 50  0001 C CNN
+F 2 "switches:SW_TH_Tactile_Omron_Fixed" H 8250 7050 50  0001 C CNN
 F 3 "" H 8250 7050 50  0001 C CNN
 	1    8250 6850
@@
 Wire Wire Line
 	6150 5250 6550 5250
-Wire Wire Line
-	6700 5350 6350 5350
-$Comp
-L pods-rescue:R R4
-U 1 1 5C082A57
-P 6350 5600
-F 0 "R4" V 6430 5600 50  0000 C CNN
-F 1 "10K" V 6350 5600 50  0000 C CNN
-F 2 "Resistor_SMD:R_0805_2012Metric_Pad1.15x1.40mm_HandSolder" V 6280 5600 50  0001 C CNN
-F 3 "" H 6350 5600 50  0001 C CNN
-	1    6350 5600
-	-1   0    0    1
-$EndComp
 $Comp
 L pods-rescue:R R5
@@
 $EndComp
 Wire Wire Line
-	6350 5450 6350 5350
-Connection ~ 6350 5350
-Wire Wire Line
-	6350 5350 6150 5350
-Wire Wire Line
 	6550 5450 6550 5250
 Connection ~ 6550 5250
@@
 	6050 5750 6050 5850
 Wire Wire Line
-	6050 5850 6350 5850
-Wire Wire Line
-	6350 5850 6350 5750
-Wire Wire Line
-	6350 5850 6550 5850
-Wire Wire Line
 	6550 5850 6550 5750
-Connection ~ 6350 5850
+Wire Wire Line
+	4300 3400 4850 3400
+Connection ~ 4300 3400
+Wire Wire Line
+	4100 4000 4100 3900
+Wire Wire Line
+	4100 3900 4850 3900
+Wire Wire Line
+	3850 4000 4100 4000
+Wire Wire Line
+	3950 3400 4300 3400
+Wire Wire Line
+	6050 5850 6550 5850
+Wire Wire Line
+	6150 5350 6700 5350
+Wire Wire Line
+	4300 3300 4300 3400
+Wire Wire Line
+	4300 3300 4850 3300
 $EndSCHEMATC
